File: Bus_switch.kicad_sch (KiCad schematic)
At the start: 15 parts, among them J3 Conn_01x04_Pin, U1 SN74CB3Q3384APW

Commit message: temp commit
Other:
- company: (none) -> MiniModucard System
- title: MMS3 Hat template small (Change Me) -> MMS3_hat_GPIO_board
Changed lines of the file:
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@@
 	(paper "A4")
 	(title_block
-		(title "MMS3 Hat template small (Change Me)")
-		(date "2026-02-25")
+		(title "MMS3_hat_GPIO_board")
+		(date "2026-02-12")
 		(rev "A")
-		(comment 1 "Made by Wojciech Szafrański")
+		(company "MiniModucard System")
+		(comment 1 "Wojciech Szafrański")
 		(comment 2 "Designed in poland")
 	)
@@
 		)
 		(instances
-			(project "MMS3_hat_templates"
+			(project "MMS3_hat_GPIO_board"
 				(path "/6596548a-44e0-46d8-8624-fd71cf4a3e17/ec6d73af-72b0-4068-85fb-cca3c5143749"
 					(reference "R7")
@@
 		)
 		(instances
-			(project "MMS3_hat_templates"
+			(project "MMS3_hat_GPIO_board"
 				(path "/6596548a-44e0-46d8-8624-fd71cf4a3e17/ec6d73af-72b0-4068-85fb-cca3c5143749"
 					(reference "R5")
@@
 		)
 		(instances
-			(project "MMS3_hat_templates"
+			(project "MMS3_hat_GPIO_board"
 				(path "/6596548a-44e0-46d8-8624-fd71cf4a3e17/ec6d73af-72b0-4068-85fb-cca3c5143749"
 					(reference "R2")
@@
 		)
 		(instances
-			(project "MMS3_hat_templates"
+			(project "MMS3_hat_GPIO_board"
 				(path "/6596548a-44e0-46d8-8624-fd71cf4a3e17/ec6d73af-72b0-4068-85fb-cca3c5143749"
 					(reference "R10")
@@
 		)
 		(instances
-			(project "MMS3_hat_templates"
+			(project "MMS3_hat_GPIO_board"
 				(path "/6596548a-44e0-46d8-8624-fd71cf4a3e17/ec6d73af-72b0-4068-85fb-cca3c5143749"
 					(reference "R9")
@@
 		)
 		(instances
-			(project "MMS3_hat_templates"
+			(project "MMS3_hat_GPIO_board"
 				(path "/6596548a-44e0-46d8-8624-fd71cf4a3e17/ec6d73af-72b0-4068-85fb-cca3c5143749"
 					(reference "#PWR038")
@@
 		)
 		(instances
-			(project "MMS3_hat_templates"
+			(project "MMS3_hat_GPIO_board"
 				(path "/6596548a-44e0-46d8-8624-fd71cf4a3e17/ec6d73af-72b0-4068-85fb-cca3c5143749"
 					(reference "#PWR047")
@@
 		)
 		(instances
-			(project "MMS3_hat_templates"
+			(project "MMS3_hat_GPIO_board"
 				(path "/6596548a-44e0-46d8-8624-fd71cf4a3e17/ec6d73af-72b0-4068-85fb-cca3c5143749"
 					(reference "#PWR051")
@@
 		)
 		(instances
-			(project "MMS3_hat_templates"
+			(project "MMS3_hat_GPIO_board"
 				(path "/6596548a-44e0-46d8-8624-fd71cf4a3e17/ec6d73af-72b0-4068-85fb-cca3c5143749"
 					(reference "#PWR036")
@@
 		)
 		(instances
-			(project "MMS3_hat_templates"
+			(project "MMS3_hat_GPIO_board"
 				(path "/6596548a-44e0-46d8-8624-fd71cf4a3e17/ec6d73af-72b0-4068-85fb-cca3c5143749"
 					(reference "J3")
@@
 		)
 		(instances
-			(project "MMS3_hat_templates"
+			(project "MMS3_hat_GPIO_board"
 				(path "/6596548a-44e0-46d8-8624-fd71cf4a3e17/ec6d73af-72b0-4068-85fb-cca3c5143749"
 					(reference "#PWR031")
@@
 		)
 		(instances
-			(project "MMS3_hat_templates"
+			(project "MMS3_hat_GPIO_board"
 				(path "/6596548a-44e0-46d8-8624-fd71cf4a3e17/ec6d73af-72b0-4068-85fb-cca3c5143749"
 					(reference "#PWR053")
@@
 		)
 		(instances
-			(project "MMS3_hat_templates"
+			(project "MMS3_hat_GPIO_board"
 				(path "/6596548a-44e0-46d8-8624-fd71cf4a3e17/ec6d73af-72b0-4068-85fb-cca3c5143749"
 					(reference "#PWR033")
@@
 		)
 		(instances
-			(project "MMS3_hat_templates"
+			(project "MMS3_hat_GPIO_board"
 				(path "/6596548a-44e0-46d8-8624-fd71cf4a3e17/ec6d73af-72b0-4068-85fb-cca3c5143749"
 					(reference "#PWR048")
@@
 		)
 		(instances
-			(project "MMS3_hat_templates"
+			(project "MMS3_hat_GPIO_board"
 				(path "/6596548a-44e0-46d8-8624-fd71cf4a3e17/ec6d73af-72b0-4068-85fb-cca3c5143749"
 					(reference "R11")
@@
 		)
 		(instances
-			(project "MMS3_hat_templates"
+			(project "MMS3_hat_GPIO_board"
 				(path "/6596548a-44e0-46d8-8624-fd71cf4a3e17/ec6d73af-72b0-4068-85fb-cca3c5143749"
 					(reference "#PWR035")
@@
 		)
 		(instances
-			(project "MMS3_hat_templates"
+			(project "MMS3_hat_GPIO_board"
 				(path "/6596548a-44e0-46d8-8624-fd71cf4a3e17/ec6d73af-72b0-4068-85fb-cca3c5143749"
 					(reference "#PWR049")
@@
 		)
 		(instances
-			(project "MMS3_hat_templates"
+			(project "MMS3_hat_GPIO_board"
 				(path "/6596548a-44e0-46d8-8624-fd71cf4a3e17/ec6d73af-72b0-4068-85fb-cca3c5143749"
 					(reference "#PWR032")
@@
 		)
 		(instances
-			(project "MMS3_hat_templates"
+			(project "MMS3_hat_GPIO_board"
 				(path "/6596548a-44e0-46d8-8624-fd71cf4a3e17/ec6d73af-72b0-4068-85fb-cca3c5143749"
 					(reference "R1")
@@
 		)
 		(instances
-			(project "MMS3_hat_templates"
+			(project "MMS3_hat_GPIO_board"
 				(path "/6596548a-44e0-46d8-8624-fd71cf4a3e17/ec6d73af-72b0-4068-85fb-cca3c5143749"
 					(reference "R6")
@@
 		)
 		(instances
-			(project "MMS3_hat_templates"
+			(project "MMS3_hat_GPIO_board"
 				(path "/6596548a-44e0-46d8-8624-fd71cf4a3e17/ec6d73af-72b0-4068-85fb-cca3c5143749"
 					(reference "D3")
@@
 		)
 		(instances
-			(project "MMS3_hat_templates"
+			(project "MMS3_hat_GPIO_board"
 				(path "/6596548a-44e0-46d8-8624-fd71cf4a3e17/ec6d73af-72b0-4068-85fb-cca3c5143749"
 					(reference "R3")
@@
 		)
 		(instances
-			(project "MMS3_hat_templates"
+			(project "MMS3_hat_GPIO_board"
 				(path "/6596548a-44e0-46d8-8624-fd71cf4a3e17/ec6d73af-72b0-4068-85fb-cca3c5143749"
 					(reference "R4")
@@
 		)
 		(instances
-			(project "MMS3_hat_templates"
+			(project "MMS3_hat_GPIO_board"
 				(path "/6596548a-44e0-46d8-8624-fd71cf4a3e17/ec6d73af-72b0-4068-85fb-cca3c5143749"
 					(reference "#PWR034")
@@
 		)
 		(instances
-			(project "MMS3_hat_templates"
+			(project "MMS3_hat_GPIO_board"
 				(path "/6596548a-44e0-46d8-8624-fd71cf4a3e17/ec6d73af-72b0-4068-85fb-cca3c5143749"
 					(reference "#PWR054")
@@
 		)
 		(instances
-			(project "MMS3_hat_templates"
+			(project "MMS3_hat_GPIO_board"
 				(path "/6596548a-44e0-46d8-8624-fd71cf4a3e17/ec6d73af-72b0-4068-85fb-cca3c5143749"
 					(reference "R8")
@@
 		)
 		(instances
-			(project "MMS3_hat_templates"
+			(project "MMS3_hat_GPIO_board"
 				(path "/6596548a-44e0-46d8-8624-fd71cf4a3e17/ec6d73af-72b0-4068-85fb-cca3c5143749"
 					(reference "#PWR037")
@@
 		)
 		(instances
-			(project "MMS3_hat_templates"
+			(project "MMS3_hat_GPIO_board"
 				(path "/6596548a-44e0-46d8-8624-fd71cf4a3e17/ec6d73af-72b0-4068-85fb-cca3c5143749"
 					(reference "#PWR052")
@@
 		)
 		(instances
-			(project "MMS3_hat_templates"
+			(project "MMS3_hat_GPIO_board"
 				(path "/6596548a-44e0-46d8-8624-fd71cf4a3e17/ec6d73af-72b0-4068-85fb-cca3c5143749"
 					(reference "U1")
@@
 		)
 		(instances
-			(project "MMS3_hat_templates"
+			(project "MMS3_hat_GPIO_board"
 				(path "/6596548a-44e0-46d8-8624-fd71cf4a3e17/ec6d73af-72b0-4068-85fb-cca3c5143749"
 					(reference "#PWR050")
@@
 		)
 		(instances
-			(project "MMS3_hat_templates"
+			(project "MMS3_hat_GPIO_board"
 				(path "/6596548a-44e0-46d8-8624-fd71cf4a3e17/ec6d73af-72b0-4068-85fb-cca3c5143749"
 					(reference "#PWR046")
@@
 		)
 		(instances
-			(project "MMS3_hat_templates"
+			(project "MMS3_hat_GPIO_board"
 				(path "/6596548a-44e0-46d8-8624-fd71cf4a3e17/ec6d73af-72b0-4068-85fb-cca3c5143749"
 					(reference "C1")
