File: ID_EEPROM.kicad_sch (KiCad schematic)
At the start: 2 parts, among them U2 M24C64

Commit message: temp commit
Other:
- company: (none) -> MiniModucard System
- title: MMS3 Hat template small (Change Me) -> MMS3_hat_GPIO_board
Changed lines of the file:
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@@
 	(paper "A4")
 	(title_block
-		(title "MMS3 Hat template small (Change Me)")
-		(date "2026-02-25")
+		(title "MMS3_hat_GPIO_board")
+		(date "2026-02-12")
 		(rev "A")
-		(comment 1 "Made by Wojciech Szafrański")
+		(company "MiniModucard System")
+		(comment 1 "Wojciech Szafrański")
 		(comment 2 "Designed in poland")
 	)
@@
 		)
 		(instances
-			(project "MMS3_hat_templates"
+			(project "MMS3_hat_GPIO_board"
 				(path "/6596548a-44e0-46d8-8624-fd71cf4a3e17/56050d79-5900-47d6-893d-3da0e8bf5810"
 					(reference "U2")
@@
 		)
 		(instances
-			(project "MMS3_hat_templates"
+			(project "MMS3_hat_GPIO_board"
 				(path "/6596548a-44e0-46d8-8624-fd71cf4a3e17/56050d79-5900-47d6-893d-3da0e8bf5810"
 					(reference "#PWR045")
@@
 		)
 		(instances
-			(project "MMS3_hat_templates"
+			(project "MMS3_hat_GPIO_board"
 				(path "/6596548a-44e0-46d8-8624-fd71cf4a3e17/56050d79-5900-47d6-893d-3da0e8bf5810"
 					(reference "#PWR044")
@@
 		)
 		(instances
-			(project "MMS3_hat_templates"
+			(project "MMS3_hat_GPIO_board"
 				(path "/6596548a-44e0-46d8-8624-fd71cf4a3e17/56050d79-5900-47d6-893d-3da0e8bf5810"
 					(reference "C2")
@@
 		)
 		(instances
-			(project "MMS3_hat_templates"
+			(project "MMS3_hat_GPIO_board"
 				(path "/6596548a-44e0-46d8-8624-fd71cf4a3e17/56050d79-5900-47d6-893d-3da0e8bf5810"
 					(reference "#PWR043")
@@
 		)
 		(instances
-			(project "MMS3_hat_templates"
+			(project "MMS3_hat_GPIO_board"
 				(path "/6596548a-44e0-46d8-8624-fd71cf4a3e17/56050d79-5900-47d6-893d-3da0e8bf5810"
 					(reference "#PWR042")
