File: Interboard_connector.kicad_sch (KiCad schematic)
At the start: 2 parts, among them J1 Chainbus in, J2 Chainbus Out

Commit message: temp commit
Other:
- company: Moducard System -> MiniModucard System
- title: MMS3 Hat template small (Change Me) -> MMS3_hat_GPIO_board
Changed lines of the file:
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@@
 	(paper "A4")
 	(title_block
-		(title "MMS3 Hat template small (Change Me)")
-		(date "2026-02-25")
+		(title "MMS3_hat_GPIO_board")
+		(date "2026-02-12")
 		(rev "A")
-		(company "Moducard System")
-		(comment 1 "Made by Wojciech Szafrański")
+		(company "MiniModucard System")
+		(comment 1 "Wojciech Szafrański")
 		(comment 2 "Designed in poland")
 	)
@@
 		)
 		(instances
-			(project "MMS3_hat_templates"
+			(project "MMS3_hat_GPIO_board"
 				(path "/6596548a-44e0-46d8-8624-fd71cf4a3e17/fdb595ff-e94b-4e80-8fe7-e7d367588ab2"
 					(reference "#PWR030")
@@
 		)
 		(instances
-			(project "MMS3_hat_templates"
+			(project "MMS3_hat_GPIO_board"
 				(path "/6596548a-44e0-46d8-8624-fd71cf4a3e17/fdb595ff-e94b-4e80-8fe7-e7d367588ab2"
 					(reference "#PWR016")
@@
 		)
 		(instances
-			(project "MMS3_hat_templates"
+			(project "MMS3_hat_GPIO_board"
 				(path "/6596548a-44e0-46d8-8624-fd71cf4a3e17/fdb595ff-e94b-4e80-8fe7-e7d367588ab2"
 					(reference "#PWR014")
@@
 		)
 		(instances
-			(project "MMS3_hat_templates"
+			(project "MMS3_hat_GPIO_board"
 				(path "/6596548a-44e0-46d8-8624-fd71cf4a3e17/fdb595ff-e94b-4e80-8fe7-e7d367588ab2"
 					(reference "#PWR041")
@@
 		)
 		(instances
-			(project "MMS3_hat_templates"
+			(project "MMS3_hat_GPIO_board"
 				(path "/6596548a-44e0-46d8-8624-fd71cf4a3e17/fdb595ff-e94b-4e80-8fe7-e7d367588ab2"
 					(reference "#PWR023")
@@
 		)
 		(instances
-			(project "MMS3_hat_templates"
+			(project "MMS3_hat_GPIO_board"
 				(path "/6596548a-44e0-46d8-8624-fd71cf4a3e17/fdb595ff-e94b-4e80-8fe7-e7d367588ab2"
 					(reference "#PWR012")
@@
 		)
 		(instances
-			(project "MMS3_hat_templates"
+			(project "MMS3_hat_GPIO_board"
 				(path "/6596548a-44e0-46d8-8624-fd71cf4a3e17/fdb595ff-e94b-4e80-8fe7-e7d367588ab2"
 					(reference "#PWR020")
@@
 		)
 		(instances
-			(project "MMS3_hat_templates"
+			(project "MMS3_hat_GPIO_board"
 				(path "/6596548a-44e0-46d8-8624-fd71cf4a3e17/fdb595ff-e94b-4e80-8fe7-e7d367588ab2"
 					(reference "#PWR04")
@@
 		)
 		(instances
-			(project "MMS3_hat_templates"
+			(project "MMS3_hat_GPIO_board"
 				(path "/6596548a-44e0-46d8-8624-fd71cf4a3e17/fdb595ff-e94b-4e80-8fe7-e7d367588ab2"
 					(reference "#PWR022")
@@
 		)
 		(instances
-			(project "MMS3_hat_templates"
+			(project "MMS3_hat_GPIO_board"
 				(path "/6596548a-44e0-46d8-8624-fd71cf4a3e17/fdb595ff-e94b-4e80-8fe7-e7d367588ab2"
 					(reference "#PWR025")
@@
 		)
 		(instances
-			(project "MMS3_hat_templates"
+			(project "MMS3_hat_GPIO_board"
 				(path "/6596548a-44e0-46d8-8624-fd71cf4a3e17/fdb595ff-e94b-4e80-8fe7-e7d367588ab2"
 					(reference "J2")
@@
 		)
 		(instances
-			(project "MMS3_hat_templates"
+			(project "MMS3_hat_GPIO_board"
 				(path "/6596548a-44e0-46d8-8624-fd71cf4a3e17/fdb595ff-e94b-4e80-8fe7-e7d367588ab2"
 					(reference "#PWR027")
@@
 		)
 		(instances
-			(project "MMS3_hat_templates"
+			(project "MMS3_hat_GPIO_board"
 				(path "/6596548a-44e0-46d8-8624-fd71cf4a3e17/fdb595ff-e94b-4e80-8fe7-e7d367588ab2"
 					(reference "#PWR09")
@@
 		)
 		(instances
-			(project "MMS3_hat_templates"
+			(project "MMS3_hat_GPIO_board"
 				(path "/6596548a-44e0-46d8-8624-fd71cf4a3e17/fdb595ff-e94b-4e80-8fe7-e7d367588ab2"
 					(reference "J1")
@@
 		)
 		(instances
-			(project "MMS3_hat_templates"
+			(project "MMS3_hat_GPIO_board"
 				(path "/6596548a-44e0-46d8-8624-fd71cf4a3e17/fdb595ff-e94b-4e80-8fe7-e7d367588ab2"
 					(reference "#PWR017")
@@
 		)
 		(instances
-			(project "MMS3_hat_templates"
+			(project "MMS3_hat_GPIO_board"
 				(path "/6596548a-44e0-46d8-8624-fd71cf4a3e17/fdb595ff-e94b-4e80-8fe7-e7d367588ab2"
 					(reference "#PWR028")
@@
 		)
 		(instances
-			(project "MMS3_hat_templates"
+			(project "MMS3_hat_GPIO_board"
 				(path "/6596548a-44e0-46d8-8624-fd71cf4a3e17/fdb595ff-e94b-4e80-8fe7-e7d367588ab2"
 					(reference "#PWR019")
@@
 		)
 		(instances
-			(project "MMS3_hat_templates"
+			(project "MMS3_hat_GPIO_board"
 				(path "/6596548a-44e0-46d8-8624-fd71cf4a3e17/fdb595ff-e94b-4e80-8fe7-e7d367588ab2"
 					(reference "#PWR029")
@@
 		)
 		(instances
-			(project "MMS3_hat_templates"
+			(project "MMS3_hat_GPIO_board"
 				(path "/6596548a-44e0-46d8-8624-fd71cf4a3e17/fdb595ff-e94b-4e80-8fe7-e7d367588ab2"
 					(reference "#PWR021")
@@
 		)
 		(instances
-			(project "MMS3_hat_templates"
+			(project "MMS3_hat_GPIO_board"
 				(path "/6596548a-44e0-46d8-8624-fd71cf4a3e17/fdb595ff-e94b-4e80-8fe7-e7d367588ab2"
 					(reference "#PWR02")
@@
 		)
 		(instances
-			(project "MMS3_hat_templates"
+			(project "MMS3_hat_GPIO_board"
 				(path "/6596548a-44e0-46d8-8624-fd71cf4a3e17/fdb595ff-e94b-4e80-8fe7-e7d367588ab2"
 					(reference "#PWR011")
@@
 		)
 		(instances
-			(project "MMS3_hat_templates"
+			(project "MMS3_hat_GPIO_board"
 				(path "/6596548a-44e0-46d8-8624-fd71cf4a3e17/fdb595ff-e94b-4e80-8fe7-e7d367588ab2"
 					(reference "#PWR018")
@@
 		)
 		(instances
-			(project "MMS3_hat_templates"
+			(project "MMS3_hat_GPIO_board"
 				(path "/6596548a-44e0-46d8-8624-fd71cf4a3e17/fdb595ff-e94b-4e80-8fe7-e7d367588ab2"
 					(reference "#PWR039")
@@
 		)
 		(instances
-			(project "MMS3_hat_templates"
+			(project "MMS3_hat_GPIO_board"
 				(path "/6596548a-44e0-46d8-8624-fd71cf4a3e17/fdb595ff-e94b-4e80-8fe7-e7d367588ab2"
 					(reference "#PWR015")
@@
 		)
 		(instances
-			(project "MMS3_hat_templates"
+			(project "MMS3_hat_GPIO_board"
 				(path "/6596548a-44e0-46d8-8624-fd71cf4a3e17/fdb595ff-e94b-4e80-8fe7-e7d367588ab2"
 					(reference "#PWR026")
@@
 		)
 		(instances
-			(project "MMS3_hat_templates"
+			(project "MMS3_hat_GPIO_board"
 				(path "/6596548a-44e0-46d8-8624-fd71cf4a3e17/fdb595ff-e94b-4e80-8fe7-e7d367588ab2"
 					(reference "#PWR05")
@@
 		)
 		(instances
-			(project "MMS3_hat_templates"
+			(project "MMS3_hat_GPIO_board"
 				(path "/6596548a-44e0-46d8-8624-fd71cf4a3e17/fdb595ff-e94b-4e80-8fe7-e7d367588ab2"
 					(reference "#PWR010")
@@
 		)
 		(instances
-			(project "MMS3_hat_templates"
+			(project "MMS3_hat_GPIO_board"
 				(path "/6596548a-44e0-46d8-8624-fd71cf4a3e17/fdb595ff-e94b-4e80-8fe7-e7d367588ab2"
 					(reference "#PWR024")
@@
 		)
 		(instances
-			(project "MMS3_hat_templates"
+			(project "MMS3_hat_GPIO_board"
 				(path "/6596548a-44e0-46d8-8624-fd71cf4a3e17/fdb595ff-e94b-4e80-8fe7-e7d367588ab2"
 					(reference "#PWR03")
@@
 		)
 		(instances
-			(project "MMS3_hat_templates"
+			(project "MMS3_hat_GPIO_board"
 				(path "/6596548a-44e0-46d8-8624-fd71cf4a3e17/fdb595ff-e94b-4e80-8fe7-e7d367588ab2"
 					(reference "#PWR013")
