File: MMS3_hat_GPIO_board.kicad_pcb (KiCad board)
At the start: 2 copper layers, 100 x 50 mm, 28 parts, among them J1 Chainbus in, J2 Chainbus Out, J3 Conn_01x04_Pin, J4 AMASS XT60 Male, J5 AMASS XT60 Female, U1 SN74CB3Q3384APW, U2 M24C64, U4 AMS1117

Commit message: temp commit
Parts:
- removed D1: M7, PCM_JLCPCB:D_SMA
- removed J4: AMASS XT60 Male, XT60:AMASS_XT60PW-M_1x02_P7.20mm_Horizontal
- removed J5: AMASS XT60 Female, XT60:AMASS_XT60PW-F_1x02_P7.20mm_Horizontal
Routing:
- net VIN_CHAINBUS: track 33.7 -> 0.76 mm
- net /Power Connector/VIN_BRD: track 32.6 -> 0.00 mm
- removed copper zone on F.Cu, net /Power Connector/VIN_BRD
