File: MMS3_hat_GPIO_board.kicad_sch (KiCad schematic)
At the start: 12 parts, among them U4 AMS1117

Commit message: temp commit
Parts:
- added J10, J4, J5, J6, J7, J8, J9: Conn_01x03_Pin, Connector_JST:JST_XH_S3B-XH-A_1x03_P2.50mm_Horizontal, symbol Connector:Conn_01x03_Pin
Connections:
- net +3V3: now also J4.3 (Pin_3)
- net GND: now also J10.1 (Pin_1), J4.1 (Pin_1), J5.1 (Pin_1), J6.1 (Pin_1), J7.1 (Pin_1), J8.1 (Pin_1), J9.1 (Pin_1)
- new net ADC: J4.2 (Pin_2)
- new net Optocoupler channel1/Output_Isolated: J9.2 (Pin_2)
- new net Optocoupler channel1/VCC: J9.3 (Pin_3)
- new net Optocoupler channel2/Output_Isolated: J10.2 (Pin_2)
- new net Optocoupler channel2/VCC: J10.3 (Pin_3)
- new net Optocoupler channel3/Output_Isolated: J7.2 (Pin_2)
- new net Optocoupler channel3/VCC: J7.3 (Pin_3)
- new net Optocoupler channel4/Output_Isolated: J8.2 (Pin_2)
- new net Optocoupler channel4/VCC: J8.3 (Pin_3)
- new net Optocoupler channel5/Output_Isolated: J5.2 (Pin_2)
- new net Optocoupler channel5/VCC: J5.3 (Pin_3)
- new net Optocoupler channel6/Output_Isolated: J6.2 (Pin_2)
- new net Optocoupler channel6/VCC: J6.3 (Pin_3)
- no-connect marks 0 -> 7
Other:
- removed sheet Power Connector
- added sheet CH32V003 (CH32V003.kicad_sch)
- added sheet GPIO Expander (TCA9535PWR_C130204.kicad_sch)
- added sheet Optocoupler channel1 (optocoupler_channel.kicad_sch)
- added sheet Optocoupler channel2 (optocoupler_channel.kicad_sch)
- added sheet Optocoupler channel3 (optocoupler_channel.kicad_sch)
- added sheet Optocoupler channel4 (optocoupler_channel.kicad_sch)
- added sheet Optocoupler channel5 (optocoupler_channel.kicad_sch)
- added sheet Optocoupler channel6 (optocoupler_channel.kicad_sch)
- added sheet VCC_selector1 (VCC_selector.kicad_sch)
- added sheet VCC_selector2 (VCC_selector.kicad_sch)
- added sheet VCC_selector3 (VCC_selector.kicad_sch)
- added sheet VCC_selector4 (VCC_selector.kicad_sch)
- added sheet VCC_selector5 (VCC_selector.kicad_sch)
- added sheet VCC_selector6 (VCC_selector.kicad_sch)
- note added: "ADC channel"
- note added: "GIVE EM A BUZZER PLZ"
- note removed: "<-- Use those connections"
- note removed: "Chainbus connector and bus switch - Do Not Modify"
- title: MMS3 Hat template small (Change Me) -> MMS3_hat_GPIO_board

Commit message: routing impossible
Parts:
- added BZ1: Buzzer, Funky_Buzzer:10_12mm_buzzer, symbol Device:Buzzer
- added R111: 0Ω, PCM_JLCPCB:R_0603, symbol PCM_JLCPCB-Resistors:0603,0Ω
Connections:
- net GND: now also R111.2
- new net: BZ1.2 (-), R111.1
- new net Buzzer: BZ1.1 (+)
- no-connect marks 7 -> 29
Other:
- sheet CH32V003 renamed CH32V003_1
- added sheet CH32V003_2 (CH32V003.kicad_sch)
- added sheet GPIO Expander1 (TCA9535PWR_C130204.kicad_sch)
- note added: "Buzzer"
- note added: "IO Channels"
- note removed: "GIVE EM A BUZZER PLZ"
- moved on the sheet: C16, C18, H1, H2, H3, H4, H5, H6, H7, H8, H9, J10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
