File: MMS3_hat_GPIO_board.kicad_sch (KiCad schematic)
At the start: 21 parts, among them J10 Conn_01x03_Pin, J4 Conn_01x03_Pin, J5 Conn_01x03_Pin, J6 Conn_01x03_Pin, J7 Conn_01x03_Pin, J8 Conn_01x03_Pin, J9 Conn_01x03_Pin, U4 AMS1117

Commit message: schematic polishing
Connections:
- no-connect marks 29 -> 15
Other:
- removed sheet CH32V003_1
- removed sheet CH32V003_2
