File: TCA9535PWR_C130204.kicad_sch (KiCad schematic)
At the start: 4 parts, among them U22 TCA9535PWR_C130204

Commit message: routing impossible
Changed lines of the file:
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@@
+		)
+	)
+	(label "D_In_5"
+		(at 0.1588 14.7957 0)
+		(effects
+			(font
+				(size 1.27 1.27)
+			)
+			(justify left bottom)
+		)
+	)
+	(label "D_Out_High_4"
+		(at 14.1288 18.6057 0)
+		(effects
+			(font
+				(size 1.27 1.27)
+			)
+			(justify left bottom)
 		)
 	)
@@
 		)
 	)
+	(label "D_Out_High_6"
+		(at 0.1588 19.8757 0)
+		(effects
+			(font
+				(size 1.27 1.27)
+			)
+			(justify left bottom)
+		)
+	)
+	(label "D_Out_High_5"
+		(at 0.1588 12.2557 0)
+		(effects
+			(font
+				(size 1.27 1.27)
+			)
+			(justify left bottom)
+		)
+	)
+	(label "D_In_4"
+		(at 14.1288 21.1457 0)
+		(effects
+			(font
+				(size 1.27 1.27)
+			)
+			(justify left bottom)
+		)
+	)
+	(label "D_Out_High_4"
+		(at 0.1588 4.6357 0)
+		(effects
+			(font
+				(size 1.27 1.27)
+			)
+			(justify left bottom)
+		)
+	)
 	(label "P17"
 		(at 104.14 87.63 180)
@@
 	(label "Chainbus.SCL"
 		(at 161.29 93.98 0)
+		(effects
+			(font
+				(size 1.27 1.27)
+			)
+			(justify left bottom)
+		)
+	)
+	(label "D_Out_Low_6"
+		(at 0.1588 17.3357 0)
+		(effects
+			(font
+				(size 1.27 1.27)
+			)
+			(justify left bottom)
+		)
+	)
+	(label "D_Out_Low_5"
+		(at 14.1288 23.6857 0)
+		(effects
+			(font
+				(size 1.27 1.27)
+			)
+			(justify left bottom)
+		)
+	)
+	(label "D_In_5"
+		(at 14.1288 28.7657 0)
+		(effects
+			(font
+				(size 1.27 1.27)
+			)
+			(justify left bottom)
+		)
+	)
+	(label "D_In_6"
+		(at 14.1288 36.3857 0)
+		(effects
+			(font
+				(size 1.27 1.27)
+			)
+			(justify left bottom)
+		)
+	)
+	(label "D_In_4"
+		(at 0.1588 7.1757 0)
+		(effects
+			(font
+				(size 1.27 1.27)
+			)
+			(justify left bottom)
+		)
+	)
+	(label "D_Out_High_5"
+		(at 14.1288 26.2257 0)
+		(effects
+			(font
+				(size 1.27 1.27)
+			)
+			(justify left bottom)
+		)
+	)
+	(label "D_Out_Low_5"
+		(at 0.1588 9.7157 0)
+		(effects
+			(font
+				(size 1.27 1.27)
+			)
+			(justify left bottom)
+		)
+	)
+	(label "D_Out_Low_4"
+		(at 0.1588 2.0957 0)
+		(effects
+			(font
+				(size 1.27 1.27)
+			)
+			(justify left bottom)
+		)
+	)
+	(label "D_Out_High_6"
+		(at 14.1288 33.8457 0)
+		(effects
+			(font
+				(size 1.27 1.27)
+			)
+			(justify left bottom)
+		)
+	)
+	(label "D_In_6"
+		(at 0.1588 22.4157 0)
+		(effects
+			(font
+				(size 1.27 1.27)
+			)
+			(justify left bottom)
+		)
+	)
+	(label "D_Out_Low_4"
+		(at 14.1288 16.0657 0)
+		(effects
+			(font
+				(size 1.27 1.27)
+			)
+			(justify left bottom)
+		)
+	)
+	(label "D_Out_Low_6"
+		(at 14.1288 31.3057 0)
 		(effects
 			(font
@@
 		(instances
 			(project "MMS3_hat_GPIO_board"
-				(path "/6596548a-44e0-46d8-8624-fd71cf4a3e17/ed54ced9-663b-4ba7-a87f-f8e4a14c3986"
+				(path "/6596548a-44e0-46d8-8624-fd71cf4a3e17/2f1cd19a-9f29-4f45-b4fa-fc3bc32e9d3a"
 					(reference "D20")
+					(unit 1)
+				)
+				(path "/6596548a-44e0-46d8-8624-fd71cf4a3e17/339cfe57-e073-474b-bfe5-4beb9a5b2966"
+					(reference "D23")
 					(unit 1)
 				)
@@
 		(instances
 			(project "MMS3_hat_GPIO_board"
-				(path "/6596548a-44e0-46d8-8624-fd71cf4a3e17/ed54ced9-663b-4ba7-a87f-f8e4a14c3986"
+				(path "/6596548a-44e0-46d8-8624-fd71cf4a3e17/2f1cd19a-9f29-4f45-b4fa-fc3bc32e9d3a"
 					(reference "#PWR0153")
+					(unit 1)
+				)
+				(path "/6596548a-44e0-46d8-8624-fd71cf4a3e17/339cfe57-e073-474b-bfe5-4beb9a5b2966"
+					(reference "#PWR0186")
 					(unit 1)
 				)
@@
 		(instances
 			(project "MMS3_hat_GPIO_board"
-				(path "/6596548a-44e0-46d8-8624-fd71cf4a3e17/ed54ced9-663b-4ba7-a87f-f8e4a14c3986"
+				(path "/6596548a-44e0-46d8-8624-fd71cf4a3e17/2f1cd19a-9f29-4f45-b4fa-fc3bc32e9d3a"
 					(reference "#PWR0151")
+					(unit 1)
+				)
+				(path "/6596548a-44e0-46d8-8624-fd71cf4a3e17/339cfe57-e073-474b-bfe5-4beb9a5b2966"
+					(reference "#PWR0184")
 					(unit 1)
 				)
@@
 		(instances
 			(project "MMS3_hat_GPIO_board"
-				(path "/6596548a-44e0-46d8-8624-fd71cf4a3e17/ed54ced9-663b-4ba7-a87f-f8e4a14c3986"
+				(path "/6596548a-44e0-46d8-8624-fd71cf4a3e17/2f1cd19a-9f29-4f45-b4fa-fc3bc32e9d3a"
 					(reference "#PWR0152")
+					(unit 1)
+				)
+				(path "/6596548a-44e0-46d8-8624-fd71cf4a3e17/339cfe57-e073-474b-bfe5-4beb9a5b2966"
+					(reference "#PWR0185")
 					(unit 1)
 				)
@@
 		(instances
 			(project "MMS3_hat_GPIO_board"
-				(path "/6596548a-44e0-46d8-8624-fd71cf4a3e17/ed54ced9-663b-4ba7-a87f-f8e4a14c3986"
+				(path "/6596548a-44e0-46d8-8624-fd71cf4a3e17/2f1cd19a-9f29-4f45-b4fa-fc3bc32e9d3a"
 					(reference "C3")
+					(unit 1)
+				)
+				(path "/6596548a-44e0-46d8-8624-fd71cf4a3e17/339cfe57-e073-474b-bfe5-4beb9a5b2966"
+					(reference "C10")
 					(unit 1)
 				)
@@
 		(instances
 			(project "MMS3_hat_GPIO_board"
-				(path "/6596548a-44e0-46d8-8624-fd71cf4a3e17/ed54ced9-663b-4ba7-a87f-f8e4a14c3986"
+				(path "/6596548a-44e0-46d8-8624-fd71cf4a3e17/2f1cd19a-9f29-4f45-b4fa-fc3bc32e9d3a"
 					(reference "#PWR0150")
+					(unit 1)
+				)
+				(path "/6596548a-44e0-46d8-8624-fd71cf4a3e17/339cfe57-e073-474b-bfe5-4beb9a5b2966"
+					(reference "#PWR0183")
 					(unit 1)
 				)
@@
 		(instances
 			(project "MMS3_hat_GPIO_board"
-				(path "/6596548a-44e0-46d8-8624-fd71cf4a3e17/ed54ced9-663b-4ba7-a87f-f8e4a14c3986"
+				(path "/6596548a-44e0-46d8-8624-fd71cf4a3e17/2f1cd19a-9f29-4f45-b4fa-fc3bc32e9d3a"
 					(reference "U22")
+					(unit 1)
+				)
+				(path "/6596548a-44e0-46d8-8624-fd71cf4a3e17/339cfe57-e073-474b-bfe5-4beb9a5b2966"
+					(reference "U25")
 					(unit 1)
 				)
@@
 		(instances
 			(project "MMS3_hat_GPIO_board"
-				(path "/6596548a-44e0-46d8-8624-fd71cf4a3e17/ed54ced9-663b-4ba7-a87f-f8e4a14c3986"
+				(path "/6596548a-44e0-46d8-8624-fd71cf4a3e17/2f1cd19a-9f29-4f45-b4fa-fc3bc32e9d3a"
 					(reference "R96")
+					(unit 1)
+				)
+				(path "/6596548a-44e0-46d8-8624-fd71cf4a3e17/339cfe57-e073-474b-bfe5-4beb9a5b2966"
+					(reference "R114")
 					(unit 1)
 				)
@@
 		(instances
 			(project "MMS3_hat_GPIO_board"
-				(path "/6596548a-44e0-46d8-8624-fd71cf4a3e17/ed54ced9-663b-4ba7-a87f-f8e4a14c3986"
+				(path "/6596548a-44e0-46d8-8624-fd71cf4a3e17/2f1cd19a-9f29-4f45-b4fa-fc3bc32e9d3a"
 					(reference "#PWR0154")
 					(unit 1)
 				)
+				(path "/6596548a-44e0-46d8-8624-fd71cf4a3e17/339cfe57-e073-474b-bfe5-4beb9a5b2966"
+					(reference "#PWR0187")
+					(unit 1)
+				)
